File: oscilador_deslocamento_fase.kicad_sch (KiCad schematic)
At the start: 40 parts, among them U1 ${SIM.PARAMS}, U2 ${SIM.PARAMS}, U3 ${SIM.PARAMS}, U4 ${SIM.PARAMS}

Commit message: updates
Parts:
- added C10, C11, C12, C13, C14, C15, C16, C9: 39n, symbol Device:C
- added C17, C18, C19: 2.2n, symbol Device:C
- added C20, C21, C22: 7u, symbol Device:C
- added L4, L5, L6: 0.045, symbol Device:L
- added R14, R16: 10.2k, symbol Device:R
- added R15, R33, R35: 11.2k, symbol Device:R
- added R17: 5.6k, symbol Device:R
- added R18, R19, R20, R23, R24, R25: 4165, symbol Device:R
- added R21: 125k, symbol Device:R
- added R22: 4309, symbol Device:R
- added R26: 142k, symbol Device:R
- added R27: 4290, symbol Device:R
- added R28, R29, R30: 5906.793948739972, symbol Device:R
- added R31: 10k, symbol Device:R
- added R32: 1k, symbol Device:R
- added R34, R36: 56k, symbol Device:R
- added U10, U5, U6, U7, U8, U9: ${SIM.PARAMS}, symbol Simulation_SPICE:OPAMP
- added V13, V14, V15, V16, V17, V18, V19, V20, V22, V23, V24, V25: 15, symbol Simulation_SPICE:VDC
Connections:
- net GND: now also C10.2, C20.2, C21.2, L5.2, L6.2, R14.2, R18.2, R19.2, R20.2, R23.2, R24.2, R25.2, R28.2, R29.2, R30.2, U10.1 (+), U6.1 (+), U7.1 (+), U8.1 (+), U9.1 (+), V13.2, V14.2, V15.1, V16.2, V17.1, V18.1, V19.2, V20.1, V22.2, V23.1, V24.2, V25.1
- net out2 renamed out2_1
- new net: C11.2, C12.1, R19.1
- new net: C12.2, C13.1, R20.1
- new net: R35.2, R36.1, U10.2 (-)
- new net: C22.2, L6.1, R36.2
- new net: C13.2, R21.1, U6.5
- new net: R21.2, R22.1, U6.2 (-)
- new net: C15.2, C16.1, R25.1
- new net: C17.2, C18.1, R29.1
- new net: C21.1, L4.2, R34.2
- new net: R26.2, R27.1, U7.2 (-)
- new net: C16.2, R26.1, U7.5
- new net: R31.2, R32.1, U8.2 (-)
- new net: C14.2, C15.1, R24.1
- new net: C18.2, C19.1, R30.1
- new net: C19.2, R31.1, U8.5
- new net: C9.2, R16.1
- new net: R16.2, U5.1 (+)
- new net: R15.2, R17.1, U5.2 (-)
- new net: R33.2, R34.1, U9.2 (-)
- new net VCC2_2: U5.3 (V+), V14.1
- new net VCC3_1: U9.3 (V+), V22.1
- new net VCC4_1: U10.3 (V+), V24.1
- new net VCC_1: U6.3 (V+), V16.1
- new net VCC_2: U7.3 (V+), V13.1
- new net VCC_3: U8.3 (V+), V19.1
- new net VEE2_2: U5.4 (V-), V15.2
- new net VEE3_1: U9.4 (V-), V23.2
- new net VEE4_1: U10.4 (V-), V25.2
- new net VEE_1: U6.4 (V-), V17.2
- new net VEE_2: U7.4 (V-), V18.2
- new net VEE_3: U8.4 (V-), V20.2
- new net out2_2: C9.1, R14.1, R15.1, R17.2, U5.5
- new net out3_1: C20.1, L4.1, R33.1, U9.5
- new net out4_1: C22.1, L5.1, R35.1, U10.5
- new net out_1: C11.1, R18.1, R22.2
- new net out_2: C14.1, R23.1, R27.2
- new net out_3: C17.1, R28.1, R32.2
- no-connect marks 1 -> 2
Other:
- moved on the sheet: C1, C2, C3, C4, C5, C6, C7, C8, L1, L2, L3, R1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
